File: IO_Bottom_Board.sch (EAGLE design)
At the start: 14 parts, among them IC1 L293D, IC2 L293D, T1 BPX81

Commit message: Add files via upload
Parts:
- R2: device rcl:R-US_0204/2V -> resistor:R-TRIMM3214W
Connections:
- new net N$23: R2.E, T1.E
- net GND: now also R2.A; no longer R2.1
- net N$21: now also R2.S; no longer R2.2, T1.E
Changed lines of the file:
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@@
 <setting verticaltext="up"/>
 </settings>
-<grid distance="0.1" unitdist="inch" unit="inch" style="lines" multiple="1" display="yes" altdistance="0.01" altunitdist="inch" altunit="inch"/>
+<grid distance="0.1" unitdist="inch" unit="inch" style="lines" multiple="1" display="no" altdistance="0.01" altunitdist="inch" altunit="inch"/>
 <layers>
 <layer number="1" name="Top" color="4" fill="1" visible="no" active="no"/>
@@
 <part name="T1" library="opto-trans-siemens" library_urn="urn:adsk.eagle:library:317" deviceset="BPX81" device="" package3d_urn="urn:adsk.eagle:package:21798/1"/>
 <part name="GND4" library="audio amplifier example" library_urn="urn:adsk.eagle:library:970892" deviceset="GND" device="" value="SUP"/>
-<part name="R2" library="rcl" library_urn="urn:adsk.eagle:library:334" deviceset="R-US_" device="0204/2V" package3d_urn="urn:adsk.eagle:package:23495/1"/>
+<part name="R2" library="resistor" library_urn="urn:adsk.eagle:library:348" deviceset="R-TRIMM" device="3214W" package3d_urn="urn:adsk.eagle:package:23729/1"/>
 </parts>
 <sheets>
@@
 </instance>
 <instance part="GND4" gate="G$1" x="132.08" y="-35.56" smashed="yes"/>
-<instance part="R2" gate="G$1" x="132.08" y="-22.86" smashed="yes" rot="R90">
-<attribute name="NAME" x="130.5814" y="-26.67" size="1.778" layer="95" rot="R90"/>
-<attribute name="VALUE" x="135.382" y="-26.67" size="1.778" layer="96" rot="R90"/>
+<instance part="R2" gate="G$1" x="132.08" y="-25.4" smashed="yes">
+<attribute name="NAME" x="126.111" y="-29.21" size="1.778" layer="95" rot="R90"/>
+<attribute name="VALUE" x="128.27" y="-29.21" size="1.778" layer="96" rot="R90"/>
 </instance>
 </instances>
@@
 <segment>
 <pinref part="GND4" gate="G$1" pin="GND"/>
-<pinref part="R2" gate="G$1" pin="1"/>
-<wire x1="132.08" y1="-35.56" x2="132.08" y2="-27.94" width="0.1524" layer="91"/>
+<wire x1="132.08" y1="-30.48" x2="132.08" y2="-35.56" width="0.1524" layer="91"/>
+<pinref part="R2" gate="G$1" pin="A"/>
 </segment>
 </net>
@@
 <net name="N$21" class="0">
 <segment>
+<pinref part="JP3" gate="B" pin="13"/>
+<wire x1="88.9" y1="25.4" x2="139.7" y2="25.4" width="0.1524" layer="91"/>
+<wire x1="139.7" y1="25.4" x2="139.7" y2="-25.4" width="0.1524" layer="91"/>
+<wire x1="137.16" y1="-25.4" x2="139.7" y2="-25.4" width="0.1524" layer="91"/>
+<pinref part="R2" gate="G$1" pin="S"/>
+</segment>
+</net>
+<net name="N$23" class="0">
+<segment>
 <pinref part="T1" gate="1" pin="E"/>
-<pinref part="JP3" gate="B" pin="13"/>
-<wire x1="132.08" y1="-12.7" x2="132.08" y2="-10.16" width="0.1524" layer="91"/>
-<wire x1="88.9" y1="25.4" x2="139.7" y2="25.4" width="0.1524" layer="91"/>
-<wire x1="139.7" y1="25.4" x2="139.7" y2="-12.7" width="0.1524" layer="91"/>
-<wire x1="139.7" y1="-12.7" x2="132.08" y2="-12.7" width="0.1524" layer="91"/>
-<pinref part="R2" gate="G$1" pin="2"/>
-<wire x1="132.08" y1="-17.78" x2="132.08" y2="-12.7" width="0.1524" layer="91"/>
-<junction x="132.08" y="-12.7"/>
-</segment>
-</net>
+<wire x1="132.08" y1="-20.32" x2="132.08" y2="-10.16" width="0.1524" layer="91"/>
+<pinref part="R2" gate="G$1" pin="E"/>
+</segment>
+</net>

Commit message: Add files via upload
Parts:
- added R3: (no value), rcl:R-US_0204/2V
- added U1: LM324PW, LM324PW:LM324PW
Connections:
- new net N$25: R2.S, U1G$1.-IN1
- net GND: now also R3.1, U1G$1.GND
- net N$21: now also U1G$1.OUT1; no longer R2.S
- net N$22: now also R2.E, U1G$1.VCC
- net N$23: now also R3.2, U1G$1.+IN1; no longer R2.E
Other:
- moved on the sheet: R2
Changed lines of the file:
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@@
 <setting verticaltext="up"/>
 </settings>
-<grid distance="0.1" unitdist="inch" unit="inch" style="lines" multiple="1" display="no" altdistance="0.01" altunitdist="inch" altunit="inch"/>
+<grid distance="0.1" unitdist="inch" unit="inch" style="lines" multiple="1" display="yes" altdistance="0.01" altunitdist="inch" altunit="inch"/>
 <layers>
 <layer number="1" name="Top" color="4" fill="1" visible="no" active="no"/>
@@
 <part name="GND4" library="audio amplifier example" library_urn="urn:adsk.eagle:library:970892" deviceset="GND" device="" value="SUP"/>
 <part name="R2" library="resistor" library_urn="urn:adsk.eagle:library:348" deviceset="R-TRIMM" device="3214W" package3d_urn="urn:adsk.eagle:package:23729/1"/>
+<part name="U1" library="LM324PW" deviceset="LM324PW" device=""/>
+<part name="R3" library="rcl" library_urn="urn:adsk.eagle:library:334" deviceset="R-US_" device="0204/2V" package3d_urn="urn:adsk.eagle:package:23495/1"/>
+<part name="GND6" library="audio amplifier example" library_urn="urn:adsk.eagle:library:970892" deviceset="GND" device="" value="SUP"/>
 </parts>
 <sheets>
@@
 </instance>
 <instance part="GND4" gate="G$1" x="132.08" y="-35.56" smashed="yes"/>
-<instance part="R2" gate="G$1" x="132.08" y="-25.4" smashed="yes">
-<attribute name="NAME" x="126.111" y="-29.21" size="1.778" layer="95" rot="R90"/>
-<attribute name="VALUE" x="128.27" y="-29.21" size="1.778" layer="96" rot="R90"/>
-</instance>
+<instance part="R2" gate="G$1" x="147.32" y="-17.78" smashed="yes">
+<attribute name="NAME" x="141.351" y="-21.59" size="1.778" layer="95" rot="R90"/>
+<attribute name="VALUE" x="143.51" y="-21.59" size="1.778" layer="96" rot="R90"/>
+</instance>
+<instance part="U1" gate="G$1" x="162.56" y="7.62" smashed="yes">
+<attribute name="NAME" x="165.10313125" y="10.798909375" size="1.780190625" layer="95"/>
+<attribute name="VALUE" x="165.103140625" y="2.53371875" size="1.7802" layer="96"/>
+</instance>
+<instance part="R3" gate="G$1" x="132.08" y="-22.86" smashed="yes" rot="R90">
+<attribute name="NAME" x="130.5814" y="-26.67" size="1.778" layer="95" rot="R90"/>
+<attribute name="VALUE" x="135.382" y="-26.67" size="1.778" layer="96" rot="R90"/>
+</instance>
+<instance part="GND6" gate="G$1" x="162.56" y="-2.54" smashed="yes"/>
 </instances>
 <busses>
@@
 <segment>
 <pinref part="GND4" gate="G$1" pin="GND"/>
-<wire x1="132.08" y1="-30.48" x2="132.08" y2="-35.56" width="0.1524" layer="91"/>
+<pinref part="R3" gate="G$1" pin="1"/>
+<wire x1="132.08" y1="-35.56" x2="132.08" y2="-33.02" width="0.1524" layer="91"/>
 <pinref part="R2" gate="G$1" pin="A"/>
+<wire x1="132.08" y1="-33.02" x2="132.08" y2="-27.94" width="0.1524" layer="91"/>
+<wire x1="147.32" y1="-22.86" x2="147.32" y2="-33.02" width="0.1524" layer="91"/>
+<wire x1="147.32" y1="-33.02" x2="132.08" y2="-33.02" width="0.1524" layer="91"/>
+<junction x="132.08" y="-33.02"/>
+</segment>
+<segment>
+<pinref part="GND6" gate="G$1" pin="GND"/>
+<pinref part="U1" gate="G$1" pin="GND"/>
+<wire x1="162.56" y1="-2.54" x2="162.56" y2="0" width="0.1524" layer="91"/>
 </segment>
 </net>
@@
 <wire x1="101.6" y1="10.16" x2="101.6" y2="2.54" width="0.1524" layer="91"/>
 <junction x="101.6" y="2.54"/>
+<wire x1="101.6" y1="10.16" x2="101.6" y2="22.86" width="0.1524" layer="91"/>
+<junction x="101.6" y="10.16"/>
+<pinref part="U1" gate="G$1" pin="VCC"/>
+<wire x1="101.6" y1="22.86" x2="147.32" y2="22.86" width="0.1524" layer="91"/>
+<wire x1="147.32" y1="22.86" x2="162.56" y2="22.86" width="0.1524" layer="91"/>
+<wire x1="162.56" y1="22.86" x2="162.56" y2="15.24" width="0.1524" layer="91"/>
+<pinref part="R2" gate="G$1" pin="E"/>
+<wire x1="147.32" y1="-12.7" x2="147.32" y2="22.86" width="0.1524" layer="91"/>
+<junction x="147.32" y="22.86"/>
 </segment>
 </net>
@@
 <segment>
 <pinref part="JP3" gate="B" pin="13"/>
-<wire x1="88.9" y1="25.4" x2="139.7" y2="25.4" width="0.1524" layer="91"/>
-<wire x1="139.7" y1="25.4" x2="139.7" y2="-25.4" width="0.1524" layer="91"/>
-<wire x1="137.16" y1="-25.4" x2="139.7" y2="-25.4" width="0.1524" layer="91"/>
+<wire x1="88.9" y1="25.4" x2="170.18" y2="25.4" width="0.1524" layer="91"/>
+<pinref part="U1" gate="G$1" pin="OUT1"/>
+<wire x1="170.18" y1="7.62" x2="170.18" y2="25.4" width="0.1524" layer="91"/>
+</segment>
+</net>
+<net name="N$23" class="0">
+<segment>
+<pinref part="R3" gate="G$1" pin="2"/>
+<pinref part="T1" gate="1" pin="E"/>
+<wire x1="132.08" y1="-17.78" x2="132.08" y2="-12.7" width="0.1524" layer="91"/>
+<pinref part="U1" gate="G$1" pin="+IN1"/>
+<wire x1="132.08" y1="-12.7" x2="132.08" y2="-10.16" width="0.1524" layer="91"/>
+<wire x1="154.94" y1="10.16" x2="142.24" y2="10.16" width="0.1524" layer="91"/>
+<wire x1="142.24" y1="10.16" x2="142.24" y2="-12.7" width="0.1524" layer="91"/>
+<wire x1="142.24" y1="-12.7" x2="132.08" y2="-12.7" width="0.1524" layer="91"/>
+<junction x="132.08" y="-12.7"/>
+</segment>
+</net>
+<net name="N$25" class="0">
+<segment>
+<pinref part="U1" gate="G$1" pin="-IN1"/>
+<wire x1="154.94" y1="5.08" x2="152.4" y2="5.08" width="0.1524" layer="91"/>
+<wire x1="152.4" y1="5.08" x2="152.4" y2="-10.16" width="0.1524" layer="91"/>
+<wire x1="152.4" y1="-10.16" x2="170.18" y2="-10.16" width="0.1524" layer="91"/>
+<wire x1="170.18" y1="-10.16" x2="170.18" y2="-17.78" width="0.1524" layer="91"/>
 <pinref part="R2" gate="G$1" pin="S"/>
-</segment>
-</net>
-<net name="N$23" class="0">
-<segment>
-<pinref part="T1" gate="1" pin="E"/>
-<wire x1="132.08" y1="-20.32" x2="132.08" y2="-10.16" width="0.1524" layer="91"/>
-<pinref part="R2" gate="G$1" pin="E"/>
-</segment>
-</net>
+<wire x1="170.18" y1="-17.78" x2="152.4" y2="-17.78" width="0.1524" layer="91"/>
+</segment>
+</net>
