File: IO_Bottom_Board.brd (EAGLE design)
At the start: 112.7 x 50.8 mm, 14 parts, among them IC1 L293D, IC2 L293D, T1 BPX81

Commit message: Add files via upload
Parts:
- R2: device rcl:0204V -> resistor:RTRIM3214W
- moved R2 12.7 mm to (73.7, 39.4)
- moved R1 5.68 mm to (64.8, 40.6)
- moved IC1 5.08 mm to (50.8, 40.6)
- moved IC2 4.02 mm to (86.4, 39.4), turned to 270 degrees
- moved D1 3.81 mm to (52.1, 54.6)
- moved T1 3.81 mm to (71.1, 54.6)
- moved JP7 1.27 mm to (114.3, 44.5)
Connections:
- new net N$23: R2.3, T1.E
- net N$21: no longer T1.E
Routing:
- net N$17: track 40.3 -> 62.6 mm
- net N$23: track 0.00 -> 19.6 mm
- net N$12: track 42.8 -> 25.1 mm
- net N$10: track 31.3 -> 15.4 mm
- net N$22: track 74.1 -> 58.3 mm, vias 0 -> 1
- net N$19: track 33.8 -> 49.1 mm
- net N$21: track 59.3 -> 48.3 mm, vias 1 -> 0
- net N$8: track 90.4 -> 79.9 mm
- net N$13: track 28.7 -> 38.8 mm
- net N$14: track 49.7 -> 39.6 mm
- net GND: track 129.4 -> 119.9 mm
- net N$11: track 18.2 -> 26.9 mm
- net N$7: track 80.9 -> 73.8 mm
- net N$4: track 85.8 -> 92.3 mm
- net N$18: track 101.3 -> 107.3 mm, vias 1 -> 0
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
Commit message: Add files via upload
Parts:
- added R3: (no value), rcl:0204V
- added U1: LM324PW, LM324PW:SOP65P640X120-14N
- moved R2 2.54 mm to (73.7, 36.8)
Connections:
- new net N$25: R2.2, U1.2
- net GND: now also R3.1, U1.11
- net N$21: now also U1.1; no longer R2.2
- net N$22: now also R2.3, U1.4
- net N$23: now also R3.2, U1.3; no longer R2.3
Routing:
- net N$5: track 29.8 -> 51.5 mm
- net N$25: track 0.00 -> 10.4 mm
- net N$4: track 92.3 -> 82.6 mm
- net GND: track 119.9 -> 129.2 mm, vias 0 -> 2
- net N$22: track 58.3 -> 67.1 mm
- net N$21: track 48.3 -> 40.6 mm
- net N$9: track 63.1 -> 55.9 mm
- net N$3: track 76.4 -> 69.9 mm
- net N$18: track 107.3 -> 113.1 mm
- net N$23: track 19.6 -> 24.8 mm
- net N$8: track 79.9 -> 83.7 mm
- net N$17: track 62.6 -> 65.0 mm
- net N$13: track 38.8 -> 40.5 mm
- net N$15: track 42.1 -> 43.4 mm
- net N$7: track 73.8 -> 72.6 mm

Commit message: Add files via upload
Parts:
- moved JP7 105.6 mm to (8.89, 38.1)
- moved JP8 105.6 mm to (114.3, 38.1)
- moved R2 21.3 mm to (94.0, 43.2)
- moved R3 10.9 mm to (59.7, 44.5)
- moved U1 9.92 mm to (81.3, 52.1)
- moved JP6 9.67 mm to (67.3, 64.8)
- moved JP5 7.41 mm to (59.7, 64.8)
- moved IC2 6.84 mm to (80.0, 36.8), turned to 0 degrees
- moved IC1 5.39 mm to (47.0, 36.8)
- moved JP1 5.24 mm to (20.3, 49.5)
- moved JP2 5.24 mm to (20.3, 31.8)
- moved JP3 5.24 mm to (102.9, 49.5)
- moved JP4 5.24 mm to (102.9, 31.8)
- moved R1 4.02 mm to (66.0, 44.5)
- moved D1 1.27 mm to (52.1, 53.3)
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Routing:
- net N$4: track 82.6 -> 35.6 mm
- net N$1: track 41.8 -> 80.9 mm
- net N$17: track 65.0 -> 30.0 mm
- net N$22: track 67.1 -> 97.7 mm, vias 1 -> 0
- net GND: track 129.2 -> 159.3 mm, vias 2 -> 0
- net N$5: track 51.5 -> 24.2 mm
- net N$3: track 69.9 -> 43.5 mm
- net N$14: track 40.1 -> 59.9 mm
- net N$2: track 48.3 -> 67.3 mm
- net N$12: track 25.1 -> 43.4 mm
- net N$16: track 33.3 -> 51.4 mm
- net N$8: track 83.7 -> 65.9 mm
- net N$10: track 15.4 -> 32.4 mm
- net N$19: track 49.3 -> 34.8 mm
- net N$21: track 40.6 -> 27.0 mm
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Other:
- board size 112.7 x 50.8 mm -> 115.2 x 55.9 mm
- board text added: "C-DAC HYD"
- board text added: "IO-BOARD-BOTTOM"
- board text removed: "CDAC-HYD"
- board text removed: "DC MOTOR"
- board text removed: "IO-BOARD BOTTOM"
- board text removed: "STEPPER MOTOR"
